File: hardware/picoslidertoy.sch (EAGLE design)
At the start: 32 parts, among them U2 RASPBERRY_PICOSMD

Commit message: old picoslidertoy sync up, but moved dev to its own repo and kicad
Parts:
- added 3V3, GND, GP6, GP7, GP8, GP9: TPTP20R, testpad:TPTP20R
- R1, R10, R11, R12, R13, R14, R15, R16, R17, R18, R19, R2, R3, R4, R5, R6, R7, R8, R9: value (none) -> 1M
- R20, R21: value (none) -> 4.7k
- SLIDER1, SLIDER2, SLIDER3: value TOUCHSLIDER36X30 -> TOUCHSLIDER36X40; device todstuff2023:TOUCHSLIDER36X30 -> todstuff2023:TOUCHSLIDER36X40
- SMDBACK2: value 13"OLED -> 13"OLEDSMDONLY; device 13oled:13"OLED -> 13oled:13"OLEDSMDONLY
- renumbered U2 to U1
Connections:
- new net N$1: GP6.TP, U1.GP6
- new net N$2: GP7.TP, U1.GP7
- new net N$3: GP9.TP, U1.GP9
- new net N$4: GP8.TP, U1.GP8
- net +3V3: now also 3V3.TP, R20.2, R21.2; no longer R16.2, R17.2
- net GND: now also GND.TP, R16.1, R17.1; no longer R20.1, R21.1
- net SCL: now also R20.1; no longer R16.1
- net SDA: now also R21.1; no longer R17.1
- net TPAD1: now also R16.2; no longer R18.2
- net TPAD2: now also R17.2; no longer R19.2
- net TPAD3: now also R18.2; no longer R20.2
- net TPAD4: now also R19.2; no longer R21.2
Other:
- moved on the sheet: R16, R17, R18, R19, R20, R21
